File: PCB/PCB_Ewine_Capteurs/PCB_Ewine.kicad_sch (KiCad schematic)
At the start: 17 parts, among them J2 Conn_2Rows-07Pins, M1 MLX90614ESF-AAA-000-TU, U1 VL53L3CXV0DH/1, U2 XC6206PxxxMR

Commit message: wifi + pcb capteur fini + start pcb motherboard
Parts:
- removed J2: Conn_2Rows-07Pins, Connector_JST:JST_XH_B7B-XH-AM_1x07_P2.50mm_Vertical, symbol Connector_Generic:Conn_2Rows-07Pins
- added J1: Conn_01x08_Pin, Connector_PinSocket_1.27mm:PinSocket_2x04_P1.27mm_Vertical, symbol Connector:Conn_01x08_Pin
- C1, C2, C3, C4, C5: footprint Capacitor_SMD:C_0805_2012Metric -> Capacitor_SMD:C_0603_1608Metric
- M1: footprint TO254P942H425-4 -> Library:TO254P942H425-4
- R1, R2, R5, R6: footprint Resistor_SMD:R_0805_2012Metric -> Resistor_SMD:R_0603_1608Metric
- R3, R4: value 4.7K -> 10K; footprint Resistor_SMD:R_0805_2012Metric -> Resistor_SMD:R_0603_1608Metric
- R7, R8: value 4.7K -> 0; footprint Resistor_SMD:R_0805_2012Metric -> Resistor_SMD:R_0603_1608Metric
- U1: footprint LGA12_STM -> Library:LGA12_STM
Connections:
- net GND_VL is gone; now on net GND: C2.2, C3.2, U1.12 (GND4), U1.2 (AVSSVCSEL), U1.3 (GND), U1.4 (GND2), U1.6 (GND3)
- net 3.3V: now also J1.6 (Pin_6)
- net 5V: now also J1.1 (Pin_1)
- net GND: now also J1.3 (Pin_3)
- net GPIO_IRQ: now also J1.7 (Pin_7)
- net SCL: now also J1.4 (Pin_4)
- net SDA: now also J1.2 (Pin_2)
- net XSHUT: now also J1.8 (Pin_8)
